File: pcb/adelheid.sch (KiCad schematic (older format))
At the start: 40 parts, among them J1 USB_B_Mini, J12 VCC, J13 D+, J14 D-, J15 GND, J2 MISO, J3 VCC, J4 SCK, J5 MOSI, J6 RES, J7 GND, J8 PF4, J9 PF5, Q1 2N7002, U1 USBLC6-2SC6, U2 ATmega32U4-AU, Y1 Crystal_GND24

Commit message: Add new plate design. Start modfying schematic
Parts:
- J1: symbol Connector:USB_B_Micro -> adelheid-rescue:USB_B_Micro-Connector
Changed lines of the file:
@@
 $EndComp
 $Comp
-L Connector:USB_B_Micro J1
+L adelheid-rescue:USB_B_Micro-Connector J1
 U 1 1 5C4B21E5
 P 1000 4800
